File: Eagle/sticky-watch-v1.5.sch (EAGLE design)
At the start: 33 parts, among them M1 ELECTRET_MICROPHON-WM-63PR, T1 BC850

Commit message: v1.5 update. I'll followup with 3d models
Parts:
- removed C6: 4.7u, rcl:C-EUC0603
- removed JP1, JP2: (no value), pinhead:PINHD-1X9
- removed R1: 4k7, rcl:R-EU_R0603
- removed RD1, RD2, RD3, RD4, RD5: 1k, rcl:R-EU_R0603
- removed T1: BC850, transistor:BC850
- added BAT+, BAT-: (no value), wirepad:1,6/0,8
- added C10, C11: 4.7u, rcl:C-EUC0603
- added CS, GND, MISO, MOSI, SCLK, VCC: TPTP10R, testpad:TPTP10R
- added LEDCHG: (no value), led:LEDSML0805
- added RCHG, RLED: 1k, rcl:R-EU_R0603
- added RPROG: 4k7, rcl:R-EU_R0603
- added U$2: MCP73831, MCP73831:MCP73831
- added U1: ATMEGA328P-AU, Atmel-ATMEGA328P-AU:ATMEGA328P-AU
- added U2: (no value), MicroUSB:USB""
- C4: value 10u -> 4.7u
- renumbered LEDD1 to LED1, LEDD2 to LED2, LEDD3 to LED3, LEDD4 to LED4, LEDD5 to LED5
Connections:
- removed net D1: JP2.2, LED1.A
- removed net D3: JP2.4, LED3.A
- removed net D5: JP2.6, LED5.A
- removed net MIC-TGL: R1.1, T1.B
- removed net MISO: ISD1700SY.MISO, JP1.8
- removed net MOSI: ISD1700SY.MOSI, JP1.7
- removed net N$12: LED4.C, RD4.2
- removed net N$8: C5.1, ISD1700SY.RESET
- removed net SCLK: ISD1700SY.SCLK, JP1.9
- removed net SS: ISD1700SY.SS, JP1.6
- new net A0: U1.PC0
- new net A1: U1.PC1
- new net A2: U1.PC2
- new net A3: U1.PC3
- new net A4/SDL: U1.PC4
- new net A5/SCL: U1.PC5
- new net D10~/SS: ISD1700SY.SS, U1.PB2
- new net D11~/MOSI: ISD1700SY.MOSI, MOSI.TP, U1.PB3
- new net D12/MISO: ISD1700SY.MISO, MISO.TP, U1.PB4
- new net D13/SCLK: ISD1700SY.SCLK, SCLK.TP, U1.PB5
- new net D3~: S1.2, S1.4, U1.PD3
- new net D5~: LED2.C, U1.PD5
- new net D6~: LED3.C, U1.PD6
- new net D9~: U1.PB1
- new net RESET: CS.TP, U1.PC6
- new net RX: U1.PD0
- new net TX: U1.PD1
- new net XTAL1: U1.PB6
- new net XTAL2: U1.PB7
- net D2: now also R4.1, S2.2, S2.4, U1.PD2; no longer JP2.3, LED2.A
- net D4: now also LED1.C, U1.PD4; no longer JP2.5, LED4.A
- net D7: now also LED4.C, U1.PD7; no longer JP1.3, S2.2, S2.4
- net D8: now also LED5.C, U1.PB0; no longer JP1.4, S1.2, S1.4
- net DGND: now also BAT-.P, C10.2, C11.2, C5.1, GND.TP, RPROG.1, U$2.VSS, U1.GND, U1.GND_2, U1.GND_3, U2.GND; no longer C5.2, C6.2, JP2.9, RD1.1, RD2.1, RD3.1, RD4.1, RD5.1, T1.E
- net N$1: now also LED1.A, LED2.A, LED3.A, LED4.A, LED5.A, RLED.2; no longer JP1.5, R1.2
- net N$10: now also C4.1; no longer C6.1
- net N$15: now also RPROG.2, U$2.PROG; no longer LED1.C, RD1.2
- net N$2: now also C10.1, RCHG.2, U$2.VDD, U2.VBUS; no longer R4.1, T1.C
- net N$4: now also LEDCHG.A, RCHG.1; no longer LED5.C, RD5.2
- net N$6: now also LEDCHG.C, U$2.STAT; no longer LED2.C, RD2.2
- net N$7: now also C5.2, U1.AREF; no longer LED3.C, RD3.2
- net VCC: now also BAT+.P, C11.1, ISD1700SY.RESET, RLED.1, U$2.VBAT, U1.AVCC, U1.VCC, U1.VCC_2, VCC.TP; no longer C4.1, JP1.1
Other:
- note added: "D3 and D2 are intterup enabled"
- note added: "make sure software cycle through led"
- moved on the sheet: C3, C4, C5
